File: saha-display.brd (EAGLE design)
At the start: 100 x 60 mm, 24 parts, among them X1 S4B-PH-SM4-TB, X2 S4B-PH-SM4-TB, X3 S8B-PH-SM4-TB, Y1 PTH-ROUND3.2-6.5ROUND, Y2 PTH-ROUND3.2-6.5ROUND, Y3 PTH-ROUND3.2-6.5ROUND, Y4 PTH-ROUND3.2-6.5ROUND

Commit message: Layout complete
Parts:
- added U$1, U$3: DAFUG, saha-display:DAFUG
- moved X2 89.8 mm to (99.0, 28.0), flipped to the bottom, turned to 90 degrees
- moved X3 75.2 mm to (50.0, 1.00), flipped to the bottom, turned to 180 degrees
- moved V4 71.5 mm to (53.0, 17.0), flipped to the bottom, turned to 90 degrees
- moved V3 70.6 mm to (55.0, 17.0), flipped to the bottom, turned to 90 degrees
- moved V2 69.7 mm to (57.0, 17.0), flipped to the bottom, turned to 90 degrees
- moved V1 68.9 mm to (59.0, 17.0), flipped to the bottom, turned to 90 degrees
- moved X1 60.1 mm to (1.00, 28.0), flipped to the bottom, turned to 270 degrees
- moved C3 56.1 mm to (60.8, 27.9), flipped to the bottom, turned to 270 degrees
- moved D1 54.7 mm to (50.0, 28.0), flipped to the bottom, turned to 90 degrees
- moved C2 53.2 mm to (62.6, 28.0), flipped to the bottom, turned to 270 degrees
- moved C1 53.1 mm to (64.6, 28.0), flipped to the bottom, turned to 270 degrees
- moved R4 52.9 mm to (27.1, 27.7), flipped to the bottom, turned to 90 degrees
- moved R5 50.9 mm to (28.9, 29.1), flipped to the bottom, turned to 270 degrees
- moved R3 48.4 mm to (62.7, 35.5), flipped to the bottom
- moved R2 44.8 mm to (62.7, 37.4), flipped to the bottom
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Connections:
- net COM0: now also D1.6
- net COM1: now also D1.7
- net COM2: now also D1.8
- net COM3: now also D1.9
- net GND: now also Y1.1, Y2.1, Y3.1, Y4.1
- net K0: now also X3.8; no longer X3.4
- net K1: now also X3.7; no longer X3.5
- net K3: now also X3.5; no longer X3.7
- net K4: now also X3.4; no longer X3.8
Routing:
- net AC: track 0.00 -> 149.5 mm
- net AD: track 0.00 -> 136.7 mm
- net AE: track 0.00 -> 136.6 mm
- net AB: track 0.00 -> 132.7 mm
- net AA: track 0.00 -> 118.4 mm
- net AF: track 0.00 -> 116.6 mm
- net AG: track 0.00 -> 115.1 mm
- net ADP: track 0.00 -> 115.1 mm
- net +5V: track 0.00 -> 113.6 mm, vias 0 -> 2
- net I2CSCL: track 0.00 -> 90.9 mm, vias 0 -> 3
- net I2CSDA: track 0.00 -> 90.6 mm, vias 0 -> 3
- net COM3: track 0.00 -> 82.0 mm, vias 0 -> 1
- net COM0: track 0.00 -> 79.5 mm, vias 0 -> 2
- net COM1: track 0.00 -> 49.0 mm, vias 0 -> 2
- net COM2: track 0.00 -> 39.0 mm
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- added copper zone on layer 1, net GND
- added copper zone on layer 16, net GND
Other:
- board size 100 x 60 mm -> 100 x 56 mm
- board text added: "+5V SDA GND SCL"
- board text added: "A B C"
- board text added: "I2C ADDRESS 0x70...0x77 1110ABC"
- board text added: "KIMMOLI 2019"
- board text added: "KS0 KS1 KS2 K4 K3 K2 K1 K0"
- board text added: "SAHA DISPLAY V1.0"
- board text added: "SCL GND SDA +5V"
