File: saha-display.sch (EAGLE design)
At the start: 24 parts, among them X1 S4B-PH-SM4-TB, X2 S4B-PH-SM4-TB, X3 S8B-PH-SM4-TB, Y1 PTH-ROUND3.2-6.5ROUND, Y2 PTH-ROUND3.2-6.5ROUND, Y3 PTH-ROUND3.2-6.5ROUND, Y4 PTH-ROUND3.2-6.5ROUND

Commit message: Layout complete
Parts:
- added U$1: DAFUG, saha-display:DAFUG
Connections:
- net COM0: now also D1.COM4
- net COM1: now also D1.COM5
- net COM2: now also D1.COM6
- net COM3: now also D1.COM7
- net GND: now also Y1.1, Y2.1, Y3.1, Y4.1
- net K0: now also X3.8; no longer X3.4
- net K1: now also X3.7; no longer X3.5
- net K3: now also X3.5; no longer X3.7
- net K4: now also X3.4; no longer X3.8
Other:
- moved on the sheet: V2, V3, V4, X3
